File: TheUntitledGoose/breadboard_adapter/hexpansion-breadboard-adapter.kicad_pcb (KiCad board)
At the start: 2 copper layers, 15.2 x 40.6 mm, 3 parts, among them J1 Conn_02x10_Counter_Clockwise, J2 Conn_01x10_Pin, J3 Conn_01x10_Pin

Commit message: Stash
Connections:
- net /AH1 renamed /HS1
- net /ALS1 renamed /LS1
- net /ALS2 renamed /LS2
- net /ALS3 renamed /LS3
- net /ALS4 renamed /LS4
- net /ALS5 renamed /LS5
- net /A_NDET renamed /DET
- net /SCL_A renamed /SCL
- net /SDA_A renamed /SDA
Changed lines of the file:
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@@
 (kicad_pcb (version 20221018) (generator pcbnew)
   (general
-    (thickness 1.0)
+    (thickness 1)
   )
   (paper "A4")
@@
   (net 0 "")
   (net 1 "/GND")
-  (net 2 "/ALS1")
-  (net 3 "/ALS2")
-  (net 4 "/SDA_A")
-  (net 5 "/SCL_A")
-  (net 6 "/A_NDET")
-  (net 7 "/ALS3")
-  (net 8 "/ALS4")
-  (net 9 "/ALS5")
-  (net 10 "/AH1")
+  (net 2 "/LS1")
+  (net 3 "/LS2")
+  (net 4 "/SDA")
+  (net 5 "/SCL")
+  (net 6 "/DET")
+  (net 7 "/LS3")
+  (net 8 "/LS4")
+  (net 9 "/LS5")
+  (net 10 "/HS1")
   (net 11 "/AH2")
   (net 12 "/PORTA_3V3")
@@
   (footprint "tildagon:SFP" (layer "F.Cu")
     (at 81.17095 57.15 90)
-    (property "Sheetfile" "tildagon-base.kicad_sch")
+    (property "Sheetfile" "hexpansion-breadboard-adapter.kicad_sch")
     (property "Sheetname" "")
     (property "ki_description" "Generic connector, double row, 02x10, counter clockwise pin numbering scheme (similar to DIP package numbering), script generated (kicad-library-utils/schlib/autogen/connector/)")
@@
       (net 1 "/GND") (pinfunction "Pin_1") (pintype "passive"))
     (pad "2" smd roundrect (at -4.1 -2.6 90) (size 2 0.5) (layers "F.Cu" "F.Paste" "F.Mask") (roundrect_rratio 0.25)
-      (net 2 "/ALS1") (pinfunction "Pin_2") (pintype "passive"))
+      (net 2 "/LS1") (pinfunction "Pin_2") (pintype "passive"))
     (pad "3" smd roundrect (at -4.1 -1.8 90) (size 2 0.5) (layers "F.Cu" "F.Paste" "F.Mask") (roundrect_rratio 0.25)
-      (net 3 "/ALS2") (pinfunction "Pin_3") (pintype "passive"))
+      (net 3 "/LS2") (pinfunction "Pin_3") (pintype "passive"))
     (pad "4" smd roundrect (at -4.1 -1 90) (size 2 0.5) (layers "F.Cu" "F.Paste" "F.Mask") (roundrect_rratio 0.25)
-      (net 4 "/SDA_A") (pinfunction "Pin_4") (pintype "passive"))
+      (net 4 "/SDA") (pinfunction "Pin_4") (pintype "passive"))
     (pad "5" smd roundrect (at -4.1 -0.2 90) (size 2 0.5) (layers "F.Cu" "F.Paste" "F.Mask") (roundrect_rratio 0.25)
-      (net 5 "/SCL_A") (pinfunction "Pin_5") (pintype "passive"))
+      (net 5 "/SCL") (pinfunction "Pin_5") (pintype "passive"))
     (pad "6" smd roundrect (at -4.1 0.6 90) (size 2 0.5) (layers "F.Cu" "F.Paste" "F.Mask") (roundrect_rratio 0.25)
-      (net 6 "/A_NDET") (pinfunction "Pin_6") (pintype "passive"))
+      (net 6 "/DET") (pinfunction "Pin_6") (pintype "passive"))
     (pad "7" smd roundrect (at -4.1 1.4 90) (size 2 0.5) (layers "F.Cu" "F.Paste" "F.Mask") (roundrect_rratio 0.25)
-      (net 7 "/ALS3") (pinfunction "Pin_7") (pintype "passive"))
+      (net 7 "/LS3") (pinfunction "Pin_7") (pintype "passive"))
     (pad "8" smd roundrect (at -4.1 2.2 90) (size 2 0.5) (layers "F.Cu" "F.Paste" "F.Mask") (roundrect_rratio 0.25)
-      (net 8 "/ALS4") (pinfunction "Pin_8") (pintype "passive"))
+      (net 8 "/LS4") (pinfunction "Pin_8") (pintype "passive"))
     (pad "9" smd roundrect (at -4.1 3 90) (size 2 0.5) (layers "F.Cu" "F.Paste" "F.Mask") (roundrect_rratio 0.25)
-      (net 9 "/ALS5") (pinfunction "Pin_9") (pintype "passive"))
+      (net 9 "/LS5") (pinfunction "Pin_9") (pintype "passive"))
     (pad "10" smd roundrect (at -4.1 3.8 90) (size 2 0.5) (layers "F.Cu" "F.Paste" "F.Mask") (roundrect_rratio 0.25)
       (net 1 "/GND") (pinfunction "Pin_10") (pintype "passive"))
@@
       (net 1 "/GND") (pinfunction "Pin_11") (pintype "passive"))
     (pad "12" smd roundrect (at 4.1 2.6 90) (size 2 0.5) (layers "F.Cu" "F.Paste" "F.Mask") (roundrect_rratio 0.25)
-      (net 10 "/AH1") (pinfunction "Pin_12") (pintype "passive"))
+      (net 10 "/HS1") (pinfunction "Pin_12") (pintype "passive"))
     (pad "13" smd roundrect (at 4.1 1.8 90) (size 2 0.5) (layers "F.Cu" "F.Paste" "F.Mask") (roundrect_rratio 0.25)
       (net 11 "/AH2") (pinfunction "Pin_13") (pintype "passive"))
@@
     (descr "Through hole straight socket strip, 1x10, 2.54mm pitch, single row (from Kicad 4.0.7), script generated")
     (tags "Through hole socket strip THT 1x10 2.54mm single row")
-    (property "Sheetfile" "tildagon-base.kicad_sch")
+    (property "Sheetfile" "hexpansion-breadboard-adapter.kicad_sch")
     (property "Sheetname" "")
     (property "ki_description" "Generic connector, single row, 01x10, script generated")
@@
       (net 1 "/GND") (pinfunction "Pin_1") (pintype "passive"))
     (pad "2" thru_hole oval (at 0 -2.54) (size 1.7 1.7) (drill 1) (layers "*.Cu" "*.Mask")
-      (net 10 "/AH1") (pinfunction "Pin_2") (pintype "passive"))
+      (net 10 "/HS1") (pinfunction "Pin_2") (pintype "passive"))
     (pad "3" thru_hole oval (at 0 -5.08) (size 1.7 1.7) (drill 1) (layers "*.Cu" "*.Mask")
       (net 11 "/AH2") (pinfunction "Pin_3") (pintype "passive"))
@@
     (descr "Through hole straight socket strip, 1x10, 2.54mm pitch, single row (from Kicad 4.0.7), script generated")
     (tags "Through hole socket strip THT 1x10 2.54mm single row")
-    (property "Sheetfile" "tildagon-base.kicad_sch")
+    (property "Sheetfile" "hexpansion-breadboard-adapter.kicad_sch")
     (property "Sheetname" "")
     (property "ki_description" "Generic connector, single row, 01x10, script generated")
@@
       (net 1 "/GND") (pinfunction "Pin_1") (pintype "passive"))
     (pad "2" thru_hole oval (at 0 -2.54) (size 1.7 1.7) (drill 1) (layers "*.Cu" "*.Mask")
-      (net 2 "/ALS1") (pinfunction "Pin_2") (pintype "passive"))
+      (net 2 "/LS1") (pinfunction "Pin_2") (pintype "passive"))
     (pad "3" thru_hole oval (at 0 -5.08) (size 1.7 1.7) (drill 1) (layers "*.Cu" "*.Mask")
-      (net 3 "/ALS2") (pinfunction "Pin_3") (pintype "passive"))
+      (net 3 "/LS2") (pinfunction "Pin_3") (pintype "passive"))
     (pad "4" thru_hole oval (at 0 -7.62) (size 1.7 1.7) (drill 1) (layers "*.Cu" "*.Mask")
-      (net 4 "/SDA_A") (pinfunction "Pin_4") (pintype "passive"))
+      (net 4 "/SDA") (pinfunction "Pin_4") (pintype "passive"))
     (pad "5" thru_hole oval (at 0 -10.16) (size 1.7 1.7) (drill 1) (layers "*.Cu" "*.Mask")
-      (net 5 "/SCL_A") (pinfunction "Pin_5") (pintype "passive"))
+      (net 5 "/SCL") (pinfunction "Pin_5") (pintype "passive"))
     (pad "6" thru_hole oval (at 0 -12.7) (size 1.7 1.7) (drill 1) (layers "*.Cu" "*.Mask")
-      (net 6 "/A_NDET") (pinfunction "Pin_6") (pintype "passive"))
+      (net 6 "/DET") (pinfunction "Pin_6") (pintype "passive"))
     (pad "7" thru_hole oval (at 0 -15.24) (size 1.7 1.7) (drill 1) (layers "*.Cu" "*.Mask")
-      (net 7 "/ALS3") (pinfunction "Pin_7") (pintype "passive"))
+      (net 7 "/LS3") (pinfunction "Pin_7") (pintype "passive"))
     (pad "8" thru_hole oval (at 0 -17.78) (size 1.7 1.7) (drill 1) (layers "*.Cu" "*.Mask")
-      (net 8 "/ALS4") (pinfunction "Pin_8") (pintype "passive"))
+      (net 8 "/LS4") (pinfunction "Pin_8") (pintype "passive"))
     (pad "9" thru_hole oval (at 0 -20.32) (size 1.7 1.7) (drill 1) (layers "*.Cu" "*.Mask")
-      (net 9 "/ALS5") (pinfunction "Pin_9") (pintype "passive"))
+      (net 9 "/LS5") (pinfunction "Pin_9") (pintype "passive"))
     (pad "10" thru_hole oval (at 0 -22.86) (size 1.7 1.7) (drill 1) (layers "*.Cu" "*.Mask")
       (net 1 "/GND") (pinfunction "Pin_10") (pintype "passive"))
