File: TheUntitledGoose/breadboard_adapter/hexpansion-breadboard-adapter.kicad_sch (KiCad schematic)
At the start: 3 parts, among them J1 Conn_02x10_Counter_Clockwise, J2 Conn_01x10_Pin, J3 Conn_01x10_Pin

Commit message: Stash
Connections:
- net AH1 renamed HS1
- net ALS1 renamed LS1
- net ALS2 renamed LS2
- net ALS3 renamed LS3
- net ALS4 renamed LS4
- net ALS5 renamed LS5
- net A_NDET renamed DET
- net SCL_A renamed SCL
- net SDA_A renamed SDA
Changed lines of the file:
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@@
     (effects (font (size 1.27 1.27)) (justify left bottom))
   )
-  (label "A_NDET" (at 59.69 41.91 180) (fields_autoplaced)
+  (label "DET" (at 59.69 41.91 180) (fields_autoplaced)
     (effects (font (size 1.27 1.27)) (justify right bottom))
   )
@@
     (effects (font (size 1.27 1.27)) (justify left))
   )
-  (hierarchical_label "ALS1" (shape bidirectional) (at 50.8 30.48 0) (fields_autoplaced)
+  (hierarchical_label "LS1" (shape bidirectional) (at 50.8 30.48 0) (fields_autoplaced)
     (effects (font (size 1.27 1.27)) (justify left))
   )
-  (hierarchical_label "ALS2" (shape bidirectional) (at 50.8 33.02 0) (fields_autoplaced)
+  (hierarchical_label "LS2" (shape bidirectional) (at 50.8 33.02 0) (fields_autoplaced)
     (effects (font (size 1.27 1.27)) (justify left))
   )
-  (hierarchical_label "ALS5" (shape bidirectional) (at 52.07 48.26 0) (fields_autoplaced)
+  (hierarchical_label "LS5" (shape bidirectional) (at 52.07 48.26 0) (fields_autoplaced)
     (effects (font (size 1.27 1.27)) (justify left))
   )
-  (hierarchical_label "ALS3" (shape bidirectional) (at 52.07 43.18 0) (fields_autoplaced)
+  (hierarchical_label "LS3" (shape bidirectional) (at 52.07 43.18 0) (fields_autoplaced)
     (effects (font (size 1.27 1.27)) (justify left))
   )
@@
     (effects (font (size 1.27 1.27)) (justify left))
   )
-  (hierarchical_label "AH1" (shape bidirectional) (at 76.2 48.26 0) (fields_autoplaced)
+  (hierarchical_label "HS1" (shape bidirectional) (at 76.2 48.26 0) (fields_autoplaced)
     (effects (font (size 1.27 1.27)) (justify left))
   )
-  (hierarchical_label "SDA_A" (shape bidirectional) (at 50.8 35.56 0) (fields_autoplaced)
+  (hierarchical_label "SDA" (shape bidirectional) (at 50.8 35.56 0) (fields_autoplaced)
     (effects (font (size 1.27 1.27)) (justify left))
   )
@@
     (effects (font (size 1.27 1.27)) (justify left))
   )
-  (hierarchical_label "SCL_A" (shape bidirectional) (at 50.8 38.1 0) (fields_autoplaced)
+  (hierarchical_label "SCL" (shape bidirectional) (at 50.8 38.1 0) (fields_autoplaced)
     (effects (font (size 1.27 1.27)) (justify left))
   )
-  (hierarchical_label "ALS4" (shape bidirectional) (at 52.07 45.72 0) (fields_autoplaced)
+  (hierarchical_label "LS4" (shape bidirectional) (at 52.07 45.72 0) (fields_autoplaced)
     (effects (font (size 1.27 1.27)) (justify left))
   )
@@
     (pin "9")
     (instances
-      (project "tildagon-base"
+      (project "hexpansion-breadboard-adapter"
         (path "/6dcb0502-87e2-4c28-9ce8-81aab8925f06"
           (reference "J3") (unit 1)
@@
     (pin "9")
     (instances
-      (project "tildagon-base"
+      (project "hexpansion-breadboard-adapter"
         (path "/6dcb0502-87e2-4c28-9ce8-81aab8925f06"
           (reference "J2") (unit 1)
@@
     (pin "8")
     (instances
-      (project "tildagon-base"
+      (project "hexpansion-breadboard-adapter"
         (path "/6dcb0502-87e2-4c28-9ce8-81aab8925f06"
           (reference "J1") (unit 1)
